Commit message: ackerman control working with joystick control

File: description/robot_core.xacro (robot description, xacro)
@@ -121,7 +121,6 @@
         <child link="left_wheel_assembly"/>
         <origin xyz="${front_wheel_offset_x} ${wheel_offset_y} 0" rpy="0 0 0" />
-        <axis xyz="0 0 -1" rpy="0 0 0" />
-        <limit effort="100" velocity="1" lower="-1" upper="1"/>
-        <dynamics damping="0.0" friction="0.0"/>
+        <axis xyz="0 0 1" rpy="0 0 0" />
+        <limit lower="-0.6" upper="0.6" velocity="1.0" effort="25"/>
     </joint>
     <!-- Front Right Steering Joint -->
@@ -188,6 +187,5 @@
         <origin xyz="${front_wheel_offset_x} -${wheel_offset_y} 0" rpy="0 0 0" />
         <axis xyz="0 0 1" rpy="0 0 0" />
-        <limit effort="100" velocity="1" lower="-1" upper="1"/>
-        <dynamics damping="0.0" friction="0.0"/>
+        <limit lower="-0.6" upper="0.6" velocity="1.0" effort="25"/>
     </joint>
     <!-- Front Right Steering Joint -->

File: description/ros2_control.xacro (robot description, xacro)
@@ -35,19 +35,21 @@
             <plugin>gazebo_ros2_control/GazeboSystem</plugin>
         </hardware>
-            <joint name="left_wheel_hinge">
-            <command_interface name="position">
-                <param name="min">-0.5236</param> <!-- -30 degrees in radians -->
-                <param name="max">0.5236</param>  <!-- 30 degrees in radians -->
+        <joint name="left_wheel_hinge">
+            <command_interface name="velocity">
+                <param name="min">-1.0</param>
+                <param name="max">1.0</param>
             </command_interface>
+            <command_interface name="position"/>
+            <state_interface name="velocity"/>
             <state_interface name="position"/>
-            <state_interface name="velocity"/>
         </joint>
         <joint name="right_wheel_hinge">
-            <command_interface name="position">
-                <param name="min">-0.5236</param> <!-- -30 degrees in radians -->
-                <param name="max">0.5236</param>  <!-- 30 degrees in radians -->
+            <command_interface name="velocity">
+                <param name="min">-1.0</param>
+                <param name="max">1.0</param>
             </command_interface>
+            <command_interface name="position"/>
+            <state_interface name="velocity"/>
             <state_interface name="position"/>
-            <state_interface name="velocity"/>
         </joint>
         <joint name="left_rear_wheel_joint">
@@ -67,4 +69,12 @@
             <state_interface name="position"/>
         </joint>
+        <joint name="front_left_rotate">
+            <!-- <command_interface name="position"/> -->
+            <state_interface name="position"/>
+        </joint>
+        <joint name="front_right_rotate">
+            <!-- <command_interface name="position"/> -->
+            <state_interface name="position"/>
+        </joint>
     </ros2_control>
     <gazebo>
